File: kc9on_anttenuator/kc9on_anttenuator.kicad_sch (KiCad schematic)
At the start: 21 parts, among them J1 9v Battery, J2 Antenna, J3 Radio, Q1 J113, SW1 OS102011MA1QS1, Y1 4.000MHz

Commit message: revising and updating to be better
Parts:
- removed RV2: 20K, Potentiometer_THT:Potentiometer_Bourns_3386F_Vertical, symbol Device:R_Potentiometer_Trim
- added R6: 4.7K, Resistor_SMD:R_1206_3216Metric, symbol Device:R
Connections:
- net at C5.1, Q1.2 (S): now also R6.2
- net at RV1.3: now also R6.1

Commit message: delete is all and start again
Parts:
- SW1: footprint BNC:SWITCH_11MA1QS1 -> Atten:SWITCH_11MA1QS1
Changed lines of the file:
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@@
 					(reference "JP1")
 					(unit 1)
-					(variant
-						(name "V2 Normal")
-					)
 				)
 			)
@@
 					(reference "C3")
 					(unit 1)
-					(variant
-						(name "V2 Normal")
-					)
 				)
 			)
@@
 					(reference "R4")
 					(unit 1)
-					(variant
-						(name "V2 Normal")
-					)
 				)
 			)
@@
 					(reference "C4")
 					(unit 1)
-					(variant
-						(name "V2 Normal")
-					)
 				)
 			)
@@
 					(reference "RV1")
 					(unit 1)
-					(variant
-						(name "V2 Normal")
-					)
 				)
 			)
@@
 					(reference "J1")
 					(unit 1)
-					(variant
-						(name "V2 Normal")
-					)
 				)
 			)
@@
 					(reference "C1")
 					(unit 1)
-					(variant
-						(name "V2 Normal")
-					)
 				)
 			)
@@
 					(reference "R3")
 					(unit 1)
-					(variant
-						(name "V2 Normal")
-					)
 				)
 			)
@@
 					(reference "J2")
 					(unit 1)
-					(variant
-						(name "V2 Normal")
-					)
 				)
 			)
@@
 					(reference "J3")
 					(unit 1)
-					(variant
-						(name "V2 Normal")
-					)
 				)
 			)
@@
 					(reference "R2")
 					(unit 1)
-					(variant
-						(name "V2 Normal")
-					)
 				)
 			)
@@
 					(reference "Y1")
 					(unit 1)
-					(variant
-						(name "V2 Normal")
-					)
 				)
 			)
@@
 					(reference "R1")
 					(unit 1)
-					(variant
-						(name "V2 Normal")
-					)
 				)
 			)
@@
 					(reference "D2")
 					(unit 1)
-					(variant
-						(name "V2 Normal")
-					)
 				)
 			)
@@
 			)
 		)
-		(property "Footprint" "BNC:SWITCH_11MA1QS1"
+		(property "Footprint" "Atten:SWITCH_11MA1QS1"
 			(at 58.42 35.56 0)
 			(hide yes)
@@
 					(reference "SW1")
 					(unit 1)
-					(variant
-						(name "V2 Normal")
-					)
 				)
 			)
@@
 					(reference "R5")
 					(unit 1)
-					(variant
-						(name "V2 Normal")
-					)
 				)
 			)
@@
 					(reference "C5")
 					(unit 1)
-					(variant
-						(name "V2 Normal")
-					)
-				)
-			)
+				)
+			)

Commit message: started version 1
Parts:
- added J4, J5: Conn_01x02_Socket, Connector_PinSocket_2.54mm:PinSocket_1x02_P2.54mm_Vertical, symbol Connector:Conn_01x02_Socket
- C2: value 220pF -> 15pf; ID CL31C221JBCNNNC -> CC1206JRNPO9BN150
- J2, J3: footprint BNC:CONN_73100-0105_MOL -> Atten:CONN_73100-0105_MOL
- JP1: now not fitted
- Q1: value J113 -> MMBF5457
- R6: value 4.7K -> 2.2K; ID RMCF1206FT4K70 -> RMCF1206FT2K20
- RV1: footprint Potentiometer_THT:Potentiometer_Bourns_PTV09A-1_Single_Vertical -> Atten:TRIM_PT01-D225D-B103; symbol Device:R_Potentiometer_Trim -> Device:R_Potentiometer_MountingPin
- SW1: value OS102011MA1QS1 -> SW_SPDT
Connections:
- net GND: now also RV1.MP (MountPin)
- net at J2.2 (Ext), J3.2 (Ext), JP1.2 (B): now also J4.2 (Pin_2), J5.1 (Pin_1)
- net at C3.2, J2.1 (In): now also J4.1 (Pin_1)
- net at C4.2, J3.1 (In): now also J5.2 (Pin_2)
Other:
- note added: "The RAW Coax symbols are meant to be used on the PVC Conduit Layout of the PCB."
- moved on the sheet: J1

Commit message: added logo n stuff
Parts:
- J1: now not fitted
Changed lines of the file:
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@@
 		(on_board yes)
 		(in_pos_files yes)
-		(dnp no)
+		(dnp yes)
 		(fields_autoplaced yes)
 		(property "Reference" "J1"
@@
 					(variant
 						(name "V2 Normal")
+						(dnp no)
 						(field
 							(name "ID")
