File: kc9on_anttenuator/kc9on_anttenuator.kicad_pcb (KiCad board)
At the start: 2 copper layers, 30 x 60 mm, 20 parts, among them J1 9v Battery, J2 Antenna, J3 Radio, Q1 J113, SW1 SW_SPDT, Y1 4.000MHz

Commit message: Nearly finished V2
Parts:
- moved R2 4.57 mm to (149.9, 119.3)
- moved C2 2.56 mm to (164.9, 111.6)
Routing:
- net Net-(Q1-S): track 0.00 -> 27.2 mm, vias 0 -> 1
- net Net-(D1-A): track 5.41 -> 9.98 mm
- net Net-(Q1-D): track 25.4 -> 22.8 mm
- net Net-(SW1-C): track 14.7 -> 16.0 mm
- net Net-(J2-Ext): track 57.0 -> 56.1 mm
- net GND: vias 0 -> 200
- added copper zone on B.Cu, net GND
- added copper zone on F.Cu, net GND

Commit message: added logo n stuff
Parts:
- added G***: LOGO, LOGO, B.Cu at (166.9, 75.6)
Other:
- board text added: "Grilled Cheese Engineering 2026 Original Design by John KC9ON Updated & Adapted by Josh KK6JDC"
- board text added: "JS"

Commit message: add more silkscreen + fixes
Routing:
- net GND: vias 200 -> 201
Other:
- board text added: "ANTENNA"
- board text added: "Grilled Cheese Engineering 2026"
- board text added: "KC9ON Attenuator V2 (Layout A) Original Design by John KC9ON Updated & Adapted by Josh KK6JDC"
- board text added: "RADIO"
- board text added: "Warning: Do NOT transmit while this device is connected to the radio"
- board text removed: "Grilled Cheese Engineering 2026 Original Design by John KC9ON Updated & Adapted by Josh KK6JDC"

Commit message: Ready for review
Parts:
- moved R4 3.56 mm to (149.1, 96.4)
- moved R6 3.56 mm to (145.6, 96.4)
- moved D1 1.35 mm to (147.0, 101.8)
- moved J2 0.25 mm to (157.0, 82.7)
- moved J3 0.25 mm to (157.0, 118.3)
Routing:
- net Net-(D2-A): track 11.1 -> 2.83 mm
- net Net-(R6-Pad1): track 5.43 -> 10.0 mm
- net Net-(R4-Pad1): track 12.4 -> 8.69 mm
- net Net-(Q1-S): track 27.2 -> 30.3 mm, vias 1 -> 2
- net Net-(D1-A): track 9.98 -> 8.52 mm
- net GND: vias 201 -> 239
Other:
- board text added: "+"
- board text added: "9V Batt"
- board text added: "ANT"
- board text added: "FoxHunt Attenuator V2 (Layout A) Original by John KC9ON Updated & Adapted by Josh KK6JDC"
- board text added: "Warning: Do NOT TX into this device. RX ONLY"
- board text removed: "ANTENNA"
- board text removed: "KC9ON Attenuator V2 (Layout A) Original Design by John KC9ON Updated & Adapted by Josh KK6JDC"
- board text removed: "Warning: Do NOT transmit while this device is connected to the radio"

Commit message: Final Version before ordering
Routing:
- net Net-(D2-A): track 2.83 -> 7.51 mm
- net GND: vias 239 -> 225
Other:
- board text added: ":)"
- board text added: "FoxHunt Offset Attenuator V2 (Layout A) Original by John KC9ON Updated & Adapted by Josh KK6JDC"
- board text removed: "FoxHunt Attenuator V2 (Layout A) Original by John KC9ON Updated & Adapted by Josh KK6JDC"
Changed lines of the file:
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@@
 		(model "C:/Users/thisi/OneDrive/Documents/FoxHunt-Offset-Attenuator/project_parts_library/PT01-D225D-B103.step"
 			(offset
-				(xyz 0 0 0)
+				(xyz 0 -0.5 0)
 			)
 			(scale
@@
 			)
 			(rotate
-				(xyz 0 0 0)
+				(xyz -0 -0 -0)
 			)
 		)
@@
 		(start 142 70.5)
 		(end 172 130.5)
-		(radius 2)
+		(radius 1.5)
 		(stroke
 			(width 0.2)
@@
 		)
 	)
+	(gr_text ":)"
+		(at 151.779 95.265 295)
+		(layer "F.SilkS")
+		(effects
+			(font
+				(size 1.15 1.15)
+				(thickness 0.275)
+				(bold yes)
+			)
+			(justify left bottom)
+		)
+	)
 	(gr_text "ANT"
 		(at 162.574 73.802 0)
@@
 		)
 	)
-	(gr_text "FoxHunt Attenuator V2 (Layout A)\n\nOriginal by John KC9ON\n\nUpdated & Adapted by Josh KK6JDC "
+	(gr_text "FoxHunt Offset Attenuator V2 (Layout A)\n\nOriginal by John KC9ON\n\nUpdated & Adapted by Josh KK6JDC "
 		(at 162.828 129.428 270)
 		(layer "B.SilkS")
@@
 	)
 	(via
-		(at 156.224 99.964)
-		(size 0.6)
-		(drill 0.3)
-		(layers "F.Cu" "B.Cu")
-		(free yes)
-		(net "GND")
-	)
-	(via
 		(at 144.032 93.868)
 		(size 0.6)
@@
 	)
 	(via
-		(at 156.224 98.44)
-		(size 0.6)
-		(drill 0.3)
-		(layers "F.Cu" "B.Cu")
-		(free yes)
-		(net "GND")
-	)
-	(via
-		(at 157.748 107.584)
-		(size 0.6)
-		(drill 0.3)
-		(layers "F.Cu" "B.Cu")
-		(free yes)
-		(net "GND")
-	)
-	(via
 		(at 144.032 109.108)
 		(size 0.6)
@@
 	)
 	(via
-		(at 157.748 106.06)
-		(size 0.6)
-		(drill 0.3)
-		(layers "F.Cu" "B.Cu")
-		(free yes)
-		(net "GND")
-	)
-	(via
 		(at 161.812 113.68)
 		(size 0.6)
@@
 	)
 	(via
-		(at 159.018 104.282)
-		(size 0.6)
-		(drill 0.3)
-		(layers "F.Cu" "B.Cu")
-		(free yes)
-		(net "GND")
-	)
-	(via
 		(at 144.032 78.628)
 		(size 0.6)
@@
 	)
 	(via
-		(at 156.224 107.584)
+		(at 159.272 102.123)
 		(size 0.6)
 		(drill 0.3)
@@
 	)
 	(via
-		(at 166.892 118.252)
+		(at 156.986 97.805)
 		(size 0.6)
 		(drill 0.3)
@@
 	)
 	(via
-		(at 151.906 94.249)
+		(at 166.892 118.252)
 		(size 0.6)
 		(drill 0.3)
@@
 	)
 	(via
-		(at 169.94 127.396)
+		(at 151.906 94.249)
 		(size 0.6)
 		(drill 0.3)
@@
 	)
 	(via
-		(at 147.08 109.108)
+		(at 169.94 127.396)
 		(size 0.6)
 		(drill 0.3)
@@
 	)
 	(via
-		(at 146.572 78.12)
+		(at 147.08 109.108)
 		(size 0.6)
 		(drill 0.3)
@@
 	)
 	(via
-		(at 158.002 99.71)
+		(at 146.572 78.12)
 		(size 0.6)
 		(drill 0.3)
@@
 	)
 	(via
-		(at 154.7 104.536)
-		(size 0.6)
-		(drill 0.3)
-		(layers "F.Cu" "B.Cu")
-		(free yes)
-		(net "GND")
-	)
-	(via
-		(at 153.176 99.964)
+		(at 154.827 104.536)
 		(size 0.6)
 		(drill 0.3)
@@
 	)
 	(via
+		(at 154.827 102.25)
+		(size 0.6)
+		(drill 0.3)
+		(layers "F.Cu" "B.Cu")
+		(free yes)
+		(net "GND")
+	)
+	(via
 		(at 163.844 119.776)
 		(size 0.6)
@@
 	)
 	(via
-		(at 154.7 101.996)
-		(size 0.6)
-		(drill 0.3)
-		(layers "F.Cu" "B.Cu")
-		(free yes)
-		(net "GND")
-	)
-	(via
 		(at 150.128 72.532)
 		(size 0.6)
@@
 	)
 	(via
-		(at 144.032 103.012)
+		(at 160.669 100.091)
 		(size 0.6)
 		(drill 0.3)
@@
 	)
 	(via
-		(at 155.97 103.3676)
+		(at 144.032 103.012)
 		(size 0.6)
 		(drill 0.3)
@@
 	)
 	(via
-		(at 160.796 106.06)
-		(size 0.6)
-		(drill 0.3)
-		(layers "F.Cu" "B.Cu")
-		(free yes)
-		(net "GND")
-	)
-	(via
 		(at 166.892 121.3)
 		(size 0.6)
@@
 	)
 	(via
-		(at 154.7 98.44)
-		(size 0.6)
-		(drill 0.3)
-		(layers "F.Cu" "B.Cu")
-		(free yes)
-		(net "GND")
-	)
-	(via
 		(at 156.986 80.66)
 		(size 0.6)
@@
 	)
 	(via
+		(at 161.177 106.314)
+		(size 0.6)
+		(drill 0.3)
+		(layers "F.Cu" "B.Cu")
+		(free yes)
+		(net "GND")
+	)
+	(via
 		(at 150.128 103.012)
 		(size 0.6)
@@
 	)
 	(via
+		(at 159.272 104.409)
+		(size 0.6)
+		(drill 0.3)
+		(layers "F.Cu" "B.Cu")
+		(free yes)
+		(net "GND")
+	)
+	(via
 		(at 163.082 125.872)
 		(size 0.6)
@@
 	)
 	(via
-		(at 157.748 103.012)
+		(at 152.795 99.837)
 		(size 0.6)
 		(drill 0.3)
@@
 	)
 	(via
-		(at 156.732 101.234)
+		(at 160.796 78.628)
 		(size 0.6)
 		(drill 0.3)
@@
 	)
 	(via
-		(at 160.796 78.628)
+		(at 153.176 87.772)
 		(size 0.6)
 		(drill 0.3)
@@
 	)
 	(via
-		(at 153.176 87.772)
+		(at 156.986 101.234)
 		(size 0.6)
 		(drill 0.3)
@@
 	)
 	(via
-		(at 157.748 84.724)
+		(at 152.541 106.314)
 		(size 0.6)
 		(drill 0.3)
@@
 	)
 	(via
-		(at 161.812 107.584)
+		(at 157.748 84.724)
 		(size 0.6)
 		(drill 0.3)
@@
 	)
 	(via
-		(at 160.796 99.964)
-		(size 0.6)
-		(drill 0.3)
-		(layers "F.Cu" "B.Cu")
-		(free yes)
-		(net "GND")
-	)
-	(via
 		(at 147.08 115.204)
 		(size 0.6)
@@
 	)
 	(via
-		(at 157.748 104.536)
-		(size 0.6)
-		(drill 0.3)
-		(layers "F.Cu" "B.Cu")
-		(free yes)
-		(net "GND")
-	)
-	(via
 		(at 169.94 81.676)
 		(size 0.6)
@@
 	)
 	(via
-		(at 158.256 101.488)
-		(size 0.6)
-		(drill 0.3)
-		(layers "F.Cu" "B.Cu")
-		(free yes)
-		(net "GND")
-	)
-	(via
 		(at 157.748 87.772)
 		(size 0.6)
@@
 	)
 	(via
-		(at 156.224 112.156)
-		(size 0.6)
-		(drill 0.3)
-		(layers "F.Cu" "B.Cu")
-		(free yes)
-		(net "GND")
-	)
-	(via
 		(at 169.94 118.252)
 		(size 0.6)
@@
 	)
 	(via
-		(at 156.224 104.536)
-		(size 0.6)
-		(drill 0.3)
-		(layers "F.Cu" "B.Cu")
-		(free yes)
-		(net "GND")
-	)
-	(via
 		(at 148.096 78.12)
 		(size 0.6)
@@
 	)
 	(via
-		(at 157.748 112.156)
-		(size 0.6)
-		(drill 0.3)
-		(layers "F.Cu" "B.Cu")
-		(free yes)
-		(net "GND")
-	)
-	(via
-		(at 153.176 106.06)
-		(size 0.6)
-		(drill 0.3)
-		(layers "F.Cu" "B.Cu")
-		(free yes)
-		(net "GND")
-	)
-	(via
 		(at 147.08 93.868)
 		(size 0.6)
@@
 	)
 	(via
-		(at 159.272 98.186)
-		(size 0.6)
-		(drill 0.3)
-		(layers "F.Cu" "B.Cu")
-		(free yes)
-		(net "GND")
-	)
-	(via
-		(at 152.16 99.456)
-		(size 0.6)
-		(drill 0.3)
-		(layers "F.Cu" "B.Cu")
-		(free yes)
-		(net "GND")
-	)
-	(via
 		(at 153.176 118.252)
 		(size 0.6)
@@
 	)
 	(via
-		(at 156.224 106.06)
+		(at 150.128 109.108)
 		(size 0.6)
 		(drill 0.3)
@@
 	)
 	(via
+		(at 159.526 97.805)
+		(size 0.6)
+		(drill 0.3)
+		(layers "F.Cu" "B.Cu")
+		(free yes)
+		(net "GND")
+	)
+	(via
 		(at 151.144 91.836)
 		(size 0.6)
@@
 	)
 	(segment
-		(start 153.176 90.272)
-		(end 153.176 93.106)
+		(start 149.493 88.788)
+		(end 150.763 90.058)
+		(width 0.2)
+		(layer "F.Cu")
+		(net "Net-(D2-A)")
+	)
+	(segment
+		(start 150.763 90.058)
+		(end 152.962 90.058)
+		(width 0.2)
+		(layer "F.Cu")
+		(net "Net-(D2-A)")
+	)
+	(segment
+		(start 152.962 90.058)
+		(end 153.176 90.272)
+		(width 0.2)
+		(layer "F.Cu")
+		(net "Net-(D2-A)")
+	)
+	(segment
+		(start 153.176 93.106)
+		(end 153.176 90.272)
+		(width 0.4)
+		(layer "F.Cu")
+		(net "Net-(D2-A)")
+	)
+	(segment
+		(start 149.112 88.788)
+		(end 149.493 88.788)
 		(width 0.2)
 		(layer "F.Cu")
